Commit message: fix bug

File: src/pixle_godzilla/urdf/pixle_godzilla.urdf (robot description, URDF)
Before this commit: robot pixle_godzilla, 7 links, 6 joints
Joints:
- joint roll_spindle: limit lower=0 upper=3.1415926536 effort=100.0 velocity=40.0 -> lower=-3.15 upper=3.15 effort=100.0 velocity=40.0

Commit message: unheallth die

File: src/pixle_godzilla/urdf/pixle_godzilla.urdf (robot description, URDF)
Before this commit: robot pixle_godzilla, 7 links, 6 joints
Joints:
- joint arm: limit lower=-2.0736 upper=1.1170107213 effort=100.0 velocity=40.0 -> lower=-2.0736 upper=0.7853981634 effort=100.0 velocity=40.0
